Commit message: Update CabinetSearch and add WaterPlants and DepthRecall-v1

File: utils/mikasa/agents/ds_fetch/fetch.urdf (robot description, URDF)
Before this commit: robot ds_fetch, 29 links, 28 joints
Joints:
- joint forearm_roll_joint: limit lower=-6.28 upper=6.28 effort=29.35 velocity=1.571 -> lower=-3.141 upper=3.141 effort=29.35 velocity=1.571
- joint upperarm_roll_joint: limit lower=-6.28 upper=6.28 effort=76.94 velocity=1.571 -> lower=-3.141 upper=3.141 effort=76.94 velocity=1.571
- joint wrist_roll_joint: limit lower=-6.28 upper=6.28 effort=7.36 velocity=2.268 -> lower=-3.141 upper=3.141 effort=7.36 velocity=2.268
